File: ev-charger-met16/ev-charger-met16.sch (KiCad schematic (older format))
At the start: 57 parts, among them J1 Screw_Terminal_01x02, J2 Conn_01x03, J3 Conn_01x15, J4 Conn_01x15, J5 Lusterklemme-6mm2-40A, J6 Lusterklemme-6mm2-40A, J7 LCD-Sure, J8 UART-Harwin4, J9 Conn_01x03, Q1 NTR2101P, Q2 MMBF170, Q3 NTR2101P, Q4 MMBF170, SW1 SW_PT65-501, SW2 SW_DPDT_x2, U1 ARDUINO-NANO, U2 HLK-PM01, U3 ebay-253052736386, U4 ACS712, U5 ebay-232542976388

Commit message: ...
Parts:
- added D5: D_Schottky, Diodes_SMD:D_SOD-323_HandSoldering, symbol D_Schottky
- added D6: D_Schottky, Diodes_SMD:D_SMA-SMB_Universal_Handsoldering, symbol D_Schottky
- added J10: Conn_02x02_Counter_Clockwise, Pin_Headers:Pin_Header_Straight_2x02_Pitch2.54mm, symbol Conn_02x02_Counter_Clockwise
- added R27: 2.74k, Resistors_SMD:R_1206_HandSoldering, symbol R
- added R28: 1.3k, Resistors_SMD:R_1206_HandSoldering, symbol R
Connections:
- wire segments 232 -> 246
Other:
- note added: "Simulate car"
- moved on the sheet: D4, J1, J2, U2
