File: ev-charger-met16/ev-charger-met16.kicad_pcb (KiCad board)
At the start: 2 copper layers, 165 x 70 mm, 65 parts, among them J1 Screw_Terminal_01x02, J2 Conn_01x03, J3 Conn_01x15, J4 Conn_01x15, J5 Lusterklemme-6mm2-40A, J6 Lusterklemme-6mm2-40A, J7 LCD-Sure, J8 UART-Harwin4, J9 Conn_01x03, Q1 NTR2101P, Q2 MMBF170, Q3 NTR2101P, Q4 MMBF170, SW1 SW_PT65-501, SW2 SW_DPDT_x2, U1 ARDUINO-NANO, U2 HLK-PM01, U3 ebay-253052736386, U4 ACS712, U5 ebay-232542976388

Commit message: ...
Parts:
- added D5: D_Schottky, Diodes_SMD:D_SOD-323_HandSoldering, F.Cu at (200.9, 86.2)
- added D6: D_Schottky, Diodes_SMD:D_SMA-SMB_Universal_Handsoldering, B.Cu at (95.6, 64.0)
- added J10: Conn_02x02_Counter_Clockwise, Pin_Headers:Pin_Header_Straight_2x02_Pitch2.54mm, F.Cu at (207.1, 89.6)
- added R27: 2.74k, Resistors_SMD:R_1206_HandSoldering, F.Cu at (206.9, 98.5)
- added R28: 1.3k, Resistors_SMD:R_1206_HandSoldering, F.Cu at (209.7, 98.5)
- moved J1 2.54 mm to (193.4, 95.0)
- moved J2 1.70 mm to (203.3, 94.7)
- moved U3 0.50 mm to (102.0, 65.0)
Connections:
- U2 pad 2: +5V -> Net-(D6-Pad2)
Routing:
- net /PE: track 0.00 -> 11.4 mm
- net Net-(D5-Pad1): track 0.00 -> 10.1 mm
- net Net-(D6-Pad2): track 0.00 -> 6.24 mm
- net Net-(J10-Pad3): track 0.00 -> 4.46 mm
- net Net-(J10-Pad4): track 0.00 -> 4.35 mm
- net +12V: track 37.3 -> 41.0 mm
- net /CP: track 62.2 -> 64.3 mm
- net -12V: track 26.6 -> 24.7 mm
- net +5V: track 185.0 -> 183.9 mm
- net GND: track 47.7 -> 48.6 mm
Other:
- board text added: "conn"
- board text added: "load"

Commit message: Revision changed to 0.1
Other:
- board text added: "EV Charger MET16 V0.1 / SX"
- board text removed: "EV Charger MET16 V1.0 / SX"
Changed lines of the file:
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@@
-(kicad_pcb (version 4) (host pcbnew 4.0.7-e2-6376~58~ubuntu16.04.1)
+(kicad_pcb (version 4) (host pcbnew 4.0.7-e2-6376~61~ubuntu18.04.1)
   (general
     (links 168)
@@
   )
   (page A4)
+  (title_block
+    (title ev-charger-met16)
+    (date 2018-05-12)
+    (rev 0.1)
+    (company Manfred.Steiner@gmx.at)
+  )
   (layers
     (0 F.Cu signal)
@@
   )
   (setup
-    (last_trace_width 0.5)
+    (last_trace_width 0.25)
     (user_trace_width 0.25)
     (user_trace_width 0.4)
@@
     (effects (font (size 1.5 1.5) (thickness 0.3)))
   )
-  (gr_text "EV Charger MET16 V1.0 / SX" (at 197.728 122.89) (layer F.SilkS)
+  (gr_text "EV Charger MET16 V0.1 / SX" (at 197.728 122.89) (layer F.SilkS)
     (effects (font (size 1.2 1.2) (thickness 0.2)))
   )
